Commit message: next steps

File: description/robot_core.xacro (robot description, xacro)
@@ -37,4 +37,7 @@
         </xacro:inertial_box>
     </link>
+    <gazebo reference="chassi_link">
+        <material>Gazebo/White</material>
+    </gazebo>
     <!-- chassi joint -->
     <joint name="chassi_joint" type='fixed'>
@@ -61,4 +64,7 @@
         </xacro:inertial_cylinder>
     </link>
+    <gazebo reference="back_left_wheel">
+        <material>Gazebo/Blue</material>
+    </gazebo>
     <!-- back left wheel joint -->
     <joint name="back_left_wheel_joint" type="continuous">
@@ -86,4 +92,7 @@
         </xacro:inertial_cylinder>
     </link>
+    <gazebo reference="back_right_wheel">
+        <material>Gazebo/Blue</material>
+    </gazebo>
     <!-- back right wheel joint -->
     <joint name="back_right_wheel_joint" type="continuous">
@@ -111,4 +120,7 @@
         </xacro:inertial_cylinder>
     </link>
+    <gazebo reference="front_left_wheel">
+        <material>Gazebo/Blue</material>
+    </gazebo>
     <!-- front left wheel joint -->
     <joint name="front_left_wheel_joint" type="continuous">
@@ -136,4 +148,7 @@
         </xacro:inertial_cylinder>
     </link>
+    <gazebo reference="front_right_wheel">
+        <material>Gazebo/Blue</material>
+    </gazebo>
     <!-- front right wheel joint -->
     <joint name="front_right_wheel_joint" type="continuous">
