Commit message: Changes in diff_drive plugin, add sonar sensors

File: description/gazebo_control.xacro (robot description, xacro)
@@ -2,17 +2,20 @@
 <robot xmlns:xacro="http://www.ros.org/wiki/xacro">
     <gazebo>
-        <plugin name="skid_steer_drive_controller" filename='libgazebo_ros_skid_steer_drive.so'>
+        <plugin name="skid_steer_drive" filename='libgazebo_ros_diff_drive.so'>
             <ros>
-                <namespace>/demo</namespace>
-                <remapping>cmd_vel:=cmd_demo</remapping>
-                <remapping>odom:=odom_demo</remapping>
+                <namespace>/</namespace>
+                <remapping>cmd_vel:=cmd_vel</remapping>
+                <remapping>odom:=odom</remapping>
             </ros>
             <!-- Wheel information -->
-            <back_left_joint>back_left_wheel_joint</back_left_joint>
-            <back_right_joint>back_right_wheel_joint</back_right_joint>
-            <front_left_joint>front_left_wheel_joint</front_left_joint>
-            <front_right_joint>front_right_wheel_joint</front_right_joint>
+            <num_wheel_pairs>2</num_wheel_pairs>
+            <left_joint>back_left_wheel_joint</left_joint>
+            <right_joint>back_right_wheel_joint</right_joint>
+            <left_joint>front_left_wheel_joint</left_joint>
+            <right_joint>front_right_wheel_joint</right_joint>
             <!-- kinematics -->
-            <wheel_separation>0.09</wheel_separation>
+            <wheel_separation>0.15</wheel_separation>
+            <wheel_separation>0.15</wheel_separation>
+            <wheel_diameter>0.06</wheel_diameter>
             <wheel_diameter>0.06</wheel_diameter>
             <!-- Limits -->
@@ -23,6 +26,7 @@
             <publish_odom_tf>true</publish_odom_tf>
             <publish_wheel_tf>true</publish_wheel_tf>
-            <odometry_frame>odom_demo</odometry_frame>
-            <robot_base_frame>chassi_link</robot_base_frame>
+            <update_rate>100.0</update_rate>
+            <odometry_frame>odom</odometry_frame>
+            <robot_base_frame>base_link</robot_base_frame>
         </plugin>
     </gazebo>

File: description/robot.urdf.xacro (robot description, xacro)
@@ -1,4 +1,6 @@
 <?xml version="1.0"?>
 <robot xmlns:xacro="http://www.ros.org/wiki/xacro"  name="robot_one">
-    <xacro:include filename="robot_core.xacro" />
+    <xacro:include filename="robot2_core.xacro" />
+    <xacro:include filename="gazebo_control.xacro"/>
+    <xacro:include filename="sonar.xacro"/>
 </robot>

File: description/robot_core.xacro (robot description, xacro)
@@ -69,5 +69,5 @@
     <!-- back left wheel joint -->
     <joint name="back_left_wheel_joint" type="continuous">
-        <parent link="base_link"/>
+        <parent link="chassi_link"/>
         <child link="back_left_wheel"/>
         <origin xyz="0 0.045 0" rpy="-${pi/2} 0 0"/>
@@ -97,5 +97,5 @@
     <!-- back right wheel joint -->
     <joint name="back_right_wheel_joint" type="continuous">
-        <parent link="base_link"/>
+        <parent link="chassi_link"/>
         <child link="back_right_wheel"/>
         <origin xyz="0 -0.045 0" rpy="${pi/2} 0 0"/>
@@ -125,5 +125,5 @@
     <!-- front left wheel joint -->
     <joint name="front_left_wheel_joint" type="continuous">
-        <parent link="base_link"/>
+        <parent link="chassi_link"/>
         <child link="front_left_wheel"/>
         <origin xyz="-0.2 0.045 0" rpy="-${pi/2} 0 0"/>
@@ -153,5 +153,5 @@
     <!-- front right wheel joint -->
     <joint name="front_right_wheel_joint" type="continuous">
-        <parent link="base_link"/>
+        <parent link="chassi_link"/>
         <child link="front_right_wheel"/>
         <origin xyz="-0.2 -0.045 0" rpy="${pi/2} 0 0"/>
