Commit message: new simulation lanch, add joystick commands

File: description/inertial_macros.xacro (robot description, xacro)
@@ -1,6 +1,5 @@
 <?xml version="1.0"?>
     <robot xmlns:xacro="http://www.ros.org/wiki/xacro">
-    <!-- Specify some standard inertial calculations https://en.wikipedia.org/wiki/List_of_moments_of_inertia -->
-    <!-- These make use of xacro's mathematical functionality -->
+    <!-- https://en.wikipedia.org/wiki/List_of_moments_of_inertia -->
     <xacro:macro name="inertial_box" params="mass x y z *origin">
         <inertial>

File: description/robot.urdf.xacro (robot description, xacro)
@@ -3,4 +3,4 @@
     <xacro:include filename="robot2_core.xacro" />
     <xacro:include filename="gazebo_control.xacro"/>
-    <xacro:include filename="sonar.xacro"/>
+    <!-- <xacro:include filename="sonar.xacro"/> -->
 </robot>

File: description/robot2_core.xacro (robot description, xacro)
@@ -26,5 +26,5 @@
             <orign xyz="0 0 0.04 " rpy="0 0 0"/>
             <geometry>
-                <box size="0.28 0.15 0.04"/>
+                <box size="0.28 0.106 0.04"/>
             </geometry>
             <material name='white'/>
@@ -33,8 +33,8 @@
             <orign xyz="0 0 0.04 " rpy="0 0 0"/>
             <geometry>
-                <box size="0.28 0.15 0.04"/>
-            </geometry>
-        </collision>
-        <xacro:inertial_box mass="1" x="0.28" y="0.15" z="0.04">
+                <box size="0.28 0.106 0.04"/>
+            </geometry>
+        </collision>
+        <xacro:inertial_box mass="1" x="0.28" y="0.106" z="0.04">
             <orign xyz="0 0 0.04 " rpy="0 0 0"/>
         </xacro:inertial_box>
@@ -74,5 +74,5 @@
         <parent link="base_link"/>
         <child link="back_left_wheel"/>
-        <origin xyz="0 0.105 0" rpy="-${pi/2} 0 0"/>
+        <origin xyz="0 0.083 0" rpy="-${pi/2} 0 0"/>
         <axis xyz="0 0 1"/>
     </joint>
@@ -102,5 +102,5 @@
         <parent link="base_link"/>
         <child link="back_right_wheel"/>
-        <origin xyz="0 -0.105 0" rpy="${pi/2} 0 0"/>
+        <origin xyz="0 -0.083 0" rpy="${pi/2} 0 0"/>
         <axis xyz="0 0 -1"/>
     </joint>
@@ -130,5 +130,5 @@
         <parent link="base_link"/>
         <child link="front_left_wheel"/>
-        <origin xyz="-0.2 0.105 0" rpy="-${pi/2} 0 0"/>
+        <origin xyz="-0.2 0.083 0" rpy="-${pi/2} 0 0"/>
         <axis xyz="0 0 1"/>
     </joint>
@@ -158,5 +158,5 @@
         <parent link="base_link"/>
         <child link="front_right_wheel"/>
-        <origin xyz="-0.2 -0.105 0" rpy="${pi/2} 0 0"/>
+        <origin xyz="-0.2 -0.083 0" rpy="${pi/2} 0 0"/>
         <axis xyz="0 0 -1"/>
     </joint>
